File: piso.kicad_pcb (KiCad board)
At the start: 2 copper layers, 101 x 76 mm, 12 parts, among them J1 PPTC041LFBN-RC, SW1 1825910-6, U2 ADG794BRQZ, U3 CD4013BMT, U4 CD4013BMT

Commit message: Updated GERBER Files
Other:
- board text added: "CLK"
- board text added: "DUAL D_FFs"
- board text added: "Din0"
- board text added: "Din1"
- board text added: "Din2"
- board text added: "Din3"
- board text added: "En"
- board text added: "I/Ps"
- board text added: "MUX"
- board text added: "O/Ps"
- board text added: "PTV"
- board text added: "RST"
Changed lines of the file:
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@@
 		(at 141.46 99.5 -90)
 		(property "Reference" "S1"
-			(at 0.175 -5.425 90)
+			(at 0 0 90)
 			(layer "F.SilkS")
 			(effects
@@
 		)
 		(property "Value" "DS04-254-2-03BK-SMT"
-			(at 0 6.46 90)
+			(at -7.5 -4.54 180)
 			(layer "F.Fab")
 			(effects
@@
 		(at 151.46 99.45 -90)
 		(property "Reference" "S2"
-			(at 0.175 -5.425 90)
+			(at 0 0 90)
 			(layer "F.SilkS")
 			(effects
@@
 			(at 0.05 -7.04 90)
 			(layer "F.Fab")
+			(hide yes)
 			(effects
 				(font
@@
 		(at 118.5 100 180)
 		(property "Reference" "SW1"
-			(at -2.3627 -3.844398 180)
+			(at 0 0 180)
 			(layer "F.SilkS")
 			(effects
@@
 		(layer "Edge.Cuts")
 	)
+	(gr_text "RST"
+		(at 139.5 108.5 90)
+		(layer "F.Cu")
+		(effects
+			(font
+				(size 1 1)
+				(thickness 0.25)
+				(bold yes)
+			)
+			(justify left bottom)
+		)
+	)
+	(gr_text "Din0"
+		(at 154 109 90)
+		(layer "F.Cu")
+		(effects
+			(font
+				(size 1 1)
+				(thickness 0.25)
+				(bold yes)
+			)
+			(justify left bottom)
+		)
+	)
+	(gr_text "CLK"
+		(at 113.5 102.5 90)
+		(layer "F.Cu")
+		(effects
+			(font
+				(size 1.5 1.5)
+				(thickness 0.3)
+				(bold yes)
+			)
+			(justify left bottom)
+		)
+	)
+	(gr_text "Din3"
+		(at 145 109 90)
+		(layer "F.Cu")
+		(effects
+			(font
+				(size 1 1)
+				(thickness 0.25)
+				(bold yes)
+			)
+			(justify left bottom)
+		)
+	)
+	(gr_text "Din1"
+		(at 152 109 90)
+		(layer "F.Cu")
+		(effects
+			(font
+				(size 1 1)
+				(thickness 0.25)
+				(bold yes)
+			)
+			(justify left bottom)
+		)
+	)
+	(gr_text "En"
+		(at 143 108 90)
+		(layer "F.Cu")
+		(effects
+			(font
+				(size 1 1)
+				(thickness 0.25)
+				(bold yes)
+			)
+			(justify left bottom)
+		)
+	)
+	(gr_text "Din2"
+		(at 149.5 109 90)
+		(layer "F.Cu")
+		(effects
+			(font
+				(size 1 1)
+				(thickness 0.25)
+				(bold yes)
+			)
+			(justify left bottom)
+		)
+	)
+	(gr_text "DUAL D_FFs\n"
+		(at 180.5 136 0)
+		(layer "B.Cu")
+		(effects
+			(font
+				(size 1.5 1.5)
+				(thickness 0.3)
+				(bold yes)
+			)
+			(justify left bottom mirror)
+		)
+	)
+	(gr_text "PTV"
+		(at 107.5 158 0)
+		(layer "B.Cu")
+		(effects
+			(font
+				(size 1.5 1.5)
+				(thickness 0.3)
+				(bold yes)
+			)
+			(justify left bottom mirror)
+		)
+	)
+	(gr_text "O/Ps"
+		(at 159 157 0)
+		(layer "B.Cu")
+		(effects
+			(font
+				(size 1.5 1.5)
+				(thickness 0.3)
+				(bold yes)
+			)
+			(justify left bottom mirror)
+		)
+	)
+	(gr_text "MUX"
+		(at 147.5 130 0)
+		(layer "B.Cu")
+		(effects
+			(font
+				(size 1.5 1.5)
+				(thickness 0.3)
+				(bold yes)
+			)
+			(justify left bottom mirror)
+		)
+	)
+	(gr_text "I/Ps\n"
+		(at 148.5 100.5 0)
+		(layer "B.Cu")
+		(effects
+			(font
+				(size 1.5 1.5)
+				(thickness 0.3)
+				(bold yes)
+			)
+			(justify left bottom mirror)
+		)
+	)
+	(gr_text "DUAL D_FFs\n"
+		(at 126.5 136 0)
+		(layer "B.Cu")
+		(effects
+			(font
+				(size 1.5 1.5)
+				(thickness 0.3)
+				(bold yes)
+			)
+			(justify left bottom mirror)
+		)
+	)
 	(segment

Commit message: Updated all files
Parts:
- added R1: RP73D1J13RBTDG, RP73D1J13RBTDG:RESC1608X50N, F.Cu at (123.0, 145.3)
- added R2: RP73D1J13RBTDG, RP73D1J13RBTDG:RESC1608X50N, F.Cu at (130.0, 143.8)
- added R3: RP73D1J13RBTDG, RP73D1J13RBTDG:RESC1608X50N, F.Cu at (138.5, 144.8)
- added R4: RP73D1J13RBTDG, RP73D1J13RBTDG:RESC1608X50N, F.Cu at (147.0, 145.0)
- added R5: RP73D1J13RBTDG, RP73D1J13RBTDG:RESC1608X50N, F.Cu at (172.0, 145.3)
- renumbered Dout to Dout1
Connections:
- D0 pad 2: D0 -> Net-(D0-A)
- D1 pad 2: D1 -> Net-(D1-A)
- D2 pad 2: D2 -> Net-(D2-A)
- D3 pad 2: D3 -> Net-(D3-A)
- Dout1 pad 2: Dout -> Net-(Dout1-A)
- U3 pad 12: Net-(U3-~{Q2}) -> unconnected-(U3-~{Q2}-Pad12)
- U3 pad 2: Net-(U3-~{Q1}) -> unconnected-(U3-~{Q1}-Pad2)
- U4 pad 12: Net-(U4-~{Q2}) -> unconnected-(U4-~{Q2}-Pad12)
- U4 pad 2: Net-(U4-~{Q1}) -> unconnected-(U4-~{Q1}-Pad2)
Routing:
- net D3: track 55.6 -> 49.6 mm, vias 2 -> 3
- net Net-(D2-A): track 0.00 -> 5.94 mm
- net Net-(D0-A): track 0.00 -> 5.18 mm
- net Net-(D1-A): track 0.00 -> 4.98 mm
- net Dout: track 34.5 -> 29.5 mm
- net Net-(D3-A): track 0.00 -> 4.44 mm
- net Net-(Dout1-A): track 0.00 -> 4.44 mm
- net D0: track 68.9 -> 64.8 mm
- net D2: track 63.6 -> 60.1 mm
- net D1: track 76.5 -> 73.2 mm
