File: piso.kicad_sch (KiCad schematic)
At the start: 16 parts, among them J1 PPTC041LFBN-RC, SW1 1825910-6, U2 ADG794BRQZ, U3 CD4013BMT, U4 CD4013BMT

Commit message: Added models used
Parts:
- removed C1, C2, C3, C4: C, symbol Device:C
Connections:
- no-connect marks 2 -> 7

Commit message: Updated all files
Parts:
- added R1, R2, R3, R4, R5: RP73D1J13RBTDG, RP73D1J13RBTDG:RESC1608X50N, symbol RP73D1J13RBTDG:RP73D1J13RBTDG
Connections:
- net D0: now also R4.2; no longer D0.2 (A)
- net D1: now also R3.2; no longer D1.2 (A)
- net D2: now also R2.2; no longer D2.2 (A)
- net D3: now also R1.2; no longer D3.2 (A)
- net Dout: now also R5.2; no longer Dout1.2 (A)
- new net: D2.2 (A), R2.1
- new net: D3.2 (A), R1.1
- new net: D0.2 (A), R4.1
- new net: D1.2 (A), R3.1
- new net: Dout1.2 (A), R5.1
Other:
- moved on the sheet: D0, D1, D2, D3, Dout1, J1, S1, S2, SW1, U2, U3, U4
